File: hardware/AGD6.07.010/AGD6.07.010.kicad_pcb (KiCad board)
At the start: 4 copper layers, 100 x 150 mm, 286 parts, among them J1001 PX_ETH GH4, J1002 SIYI_ETH GH4, J1003 CAMF_ETH GH4, J1004 AI_ETH1 GH4, J1005 SERVICE_ETH GH4, J1006 AI_ETH2 GH4, J1007 ETH_SWITCH_MODULE 2x13, J1008 CAMD_ETH GH4, J101 PDB_14S XT30, J202 AI_POWER_12V XT30, J301 PX_CAN1 GH4, J302 PX_CAN2 GH4, J303 PX_TELEM1 SIYI GH6, J304 PX_TELEM2 AI GH6, J305 PX_TELEM3 RADAR GH6, J306 PX_I2C GH4, J307 PX_AD&IO GH8, J308 PX_RC_IN GH3, J309 PX_MAIN 1-8, J310 PX_AUX 1-8, J311 FTS GH3, J312 MODE_SWITCH + LID/BATT_LATCH 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, J401 CAN1 ESC CHAIN START GH4, J402 CAN1 ESC CHAIN RETURN GH4, J407 PM08-CAN GH4, J408 BMS CAN GH4, J409 REMOTE_ID GH4, J410 GNSS2 (резерв) GH4, J411 OBSTACLE_1 GH4, J412 OBSTACLE_2 GH4, J413 SPRAY_SENSORS GH8 (давл./уров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, J421 ESC1-6 PWM backup GH8, J501 SIYI_PWR XT30, J502 SIYI_DATA GH5, J503 RADAR_US-D1 GH4, J504 GNSS_PPS GH2, J601 AI_SIGNALS GH8, J602 AI_OFF_SWITCH GH2, J603 SERVICE USB-C, J604 AI_USB GH4, J701 TEMP_AI_HEATSINK GH4, J702 TEMP_AIR GH4, J801 VALVE1 XH2, J802 VALVE2 XH2, J803 LIGHTS XH2, J804 FAN XH2, J805 HEATER XH2, J806 PUMP_PWM + CAM_TRIG GH4, J901 CAM_FRONT_PWR XH2, J902 CAM_DOWN_PWR XH2, Q101 100V N-MOSFET >=40A D2PAK (на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, Q201 40V N-MOSFET >=40A D2PAK (нап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, Q801 AO3400A, Q802 AO3401A, Q803 AO3400A, Q804 AO3400A, U101 LM5069MM-1, U102 INA228AIDGSR, U201 TPS62133RGTR, U202 AP2112K-3.3TRG1, U203 LM5069MM-2, U204 INA228AIDGSR, U205 INA228AIDGSR, U501 TPD4E05U06DQA, U502 TPD4E05U06DQA, U602 TPD4E05U06DQA, U603 USBLC6-2SC6, U701 TPS3430WDRC, U702 TMP117AIDRVR, U703 SHT40-AD1B, U704 TPD4E05U06DQA, U801 BTS5030-1EJA, U802 BTS5030-1EJA, U803 BTS5030-1EJA, U804 ADS1115IDGSR

Commit message: AGD6.07.010: close 24 more connections with an external grid router
Board geometry is exported from KiCad and routed on a 0.1 mm grid
(numpy/scipy distance transforms, net-class clearances, keepouts);
every new segment is re-checked by KiCad DRC and violators removed.
Unrouted connections 66 -> 42 with no DRC errors. Adds rule
HV_14S_pads (0.2 mm, IPC-2221B B4 with mandatory coating) so escapes
from fine-pitch 14S ICs are possible; tracks and pours keep 0.3 mm.

Co-Authored-By: Claude Opus 5.5 <noreply@anthropic.com>
Claude-Session: https://claude.ai/code/session_01Qk7uTKdi6YbndB9fGuguYV
Routing:
- net /ETHERNET/E3_TXP: track 0.00 -> 131.8 mm, vias 0 -> 7
- net +12V: track 190.9 -> 297.9 mm, vias 13 -> 20
- net /ETHERNET/E1_TXN: track 0.00 -> 95.2 mm, vias 0 -> 2
- net /ETHERNET/E1_TXP: track 0.00 -> 84.0 mm, vias 0 -> 1
- net /POWER_CONVERSION/VIN_AI_F: track 5.48 -> 51.6 mm, vias 1 -> 3
- net /VIN_PROT: track 141.9 -> 178.7 mm, vias 2 -> 5
- net /POWER_INPUT_14S/VIN_RAW: track 8.71 -> 42.2 mm, vias 1 -> 2
- net /POWER_CONVERSION/V12_RAW: track 11.8 -> 36.6 mm, vias 2 -> 3
- net /POWER_INPUT_14S/VIN_F: track 45.7 -> 66.8 mm, vias 5 -> 8
- net /LOAD_SWITCHES_12V/V12_FAN: track 5.99 -> 18.9 mm
- net GND: track 436.7 -> 442.6 mm, vias 374 -> 379
- net /I2C_SDA: track 109.9 -> 115.4 mm, vias 9 -> 10
- net /POWER_CONVERSION/V12_ALERT_N: track 2.78 -> 7.84 mm, vias 2 -> 3
- net /I2C_SCL: track 119.5 -> 123.6 mm
- net /LOAD_SWITCHES_12V/OUT1: track 10.2 -> 12.7 mm, vias 1 -> 3
