File: hardware/AGD6.07.010/AGD6.07.010.kicad_pcb (KiCad board)
At the start: 4 copper layers, 100 x 150 mm, 286 parts, among them J1001 PX_ETH GH4, J1002 SIYI_ETH GH4, J1003 CAMF_ETH GH4, J1004 AI_ETH1 GH4, J1005 SERVICE_ETH GH4, J1006 AI_ETH2 GH4, J1007 ETH_SWITCH_MODULE 2x13, J1008 CAMD_ETH GH4, J101 PDB_14S XT30, J202 AI_POWER_12V XT30, J301 PX_CAN1 GH4, J302 PX_CAN2 GH4, J303 PX_TELEM1 SIYI GH6, J304 PX_TELEM2 AI GH6, J305 PX_TELEM3 RADAR GH6, J306 PX_I2C GH4, J307 PX_AD&IO GH8, J308 PX_RC_IN GH3, J309 PX_MAIN 1-8, J310 PX_AUX 1-8, J311 FTS GH3, J312 MODE_SWITCH + LID/BATT_LATCH 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, J401 CAN1 ESC CHAIN START GH4, J402 CAN1 ESC CHAIN RETURN GH4, J407 PM08-CAN GH4, J408 BMS CAN GH4, J409 REMOTE_ID GH4, J410 GNSS2 (резерв) GH4, J411 OBSTACLE_1 GH4, J412 OBSTACLE_2 GH4, J413 SPRAY_SENSORS GH8 (давл./уров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, J421 ESC1-6 PWM backup GH8, J501 SIYI_PWR XT30, J502 SIYI_DATA GH5, J503 RADAR_US-D1 GH4, J504 GNSS_PPS GH2, J601 AI_SIGNALS GH8, J602 AI_OFF_SWITCH GH2, J603 SERVICE USB-C, J604 AI_USB GH4, J701 TEMP_AI_HEATSINK GH4, J702 TEMP_AIR GH4, J801 VALVE1 XH2, J802 VALVE2 XH2, J803 LIGHTS XH2, J804 FAN XH2, J805 HEATER XH2, J806 PUMP_PWM + CAM_TRIG GH4, J901 CAM_FRONT_PWR XH2, J902 CAM_DOWN_PWR XH2, Q101 100V N-MOSFET >=40A D2PAK (на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, Q201 40V N-MOSFET >=40A D2PAK (нап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, Q801 AO3400A, Q802 AO3401A, Q803 AO3400A, Q804 AO3400A, U101 LM5069MM-1, U102 INA228AIDGSR, U201 TPS62133RGTR, U202 AP2112K-3.3TRG1, U203 LM5069MM-2, U204 INA228AIDGSR, U205 INA228AIDGSR, U501 TPD4E05U06DQA, U502 TPD4E05U06DQA, U602 TPD4E05U06DQA, U603 USBLC6-2SC6, U701 TPS3430WDRC, U702 TMP117AIDRVR, U703 SHT40-AD1B, U704 TPD4E05U06DQA, U801 BTS5030-1EJA, U802 BTS5030-1EJA, U803 BTS5030-1EJA, U804 ADS1115IDGSR

Commit message: AGD6.07.010: AI computer RK3588 - PS202 = TEP 75-4812WI, RS201 10 mOhm, docs and outputs updated
Co-Authored-By: Claude Opus 5.5 <noreply@anthropic.com>
Claude-Session: https://claude.ai/code/session_01Qk7uTKdi6YbndB9fGuguYV
Parts:
- PS202: value DATA_REQUIRED изолир. 48V->12V >=100W -> TRACO TEP 75-4812WI
- RS201: value 5m 1W -> 10m 1W
Changed lines of the file:
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@@
 			)
 		)
-		(property "Value" "DATA_REQUIRED изолир. 48V->12V >=100W"
+		(property "Value" "TRACO TEP 75-4812WI"
 			(at 0 14.2 0)
 			(layer "F.Fab")
@@
 			)
 		)
-		(property "Value" "5m 1W"
+		(property "Value" "10m 1W"
 			(at 0 2.63 0)
 			(layer "F.Fab")
