File: hardware/AGD6.07.010/can_and_sensors.kicad_sch (KiCad schematic)
At the start: 0 parts

Commit message: Draw full AGD6.07.010 schematic per integrated_avionics_board spec
All ten sheets now carry components: 14S input with hot-swap and power
monitor, 12/5/3.3 V rails and a separate 12 V AI channel with soft-start
and current telemetry, Pixhawk connectors, CAN1/CAN2 hub with chokes,
ESD and switchable termination, sensor conditioning, SIYI and radar,
AI interface and watchdog, protected 12 V switches with diagnostics,
fan/heater control, cameras and Ethernet. Open choices are recorded in
DECISIONS.md; datasheet-dependent values are flagged CHECK_DATASHEET.

ERC: no errors. All 752 intended pin connections match the KiCad netlist.

Co-Authored-By: Claude Opus 5.5 <noreply@anthropic.com>
Claude-Session: https://claude.ai/code/session_01Qk7uTKdi6YbndB9fGuguYV
Parts:
- added C411, C421: 100n, Capacitor_SMD:C_0402_1005Metric, symbol Device:C
- added C431: 1n, Capacitor_SMD:C_0402_1005Metric, symbol Device:C
- added D411, D421: NUP2105L, Package_TO_SOT_SMD:SOT-23, symbol Power_Protection:NUP2105L
- added D412, D422, D432: ESD9B5.0ST5G, Diode_SMD:D_SOD-923, symbol Diode:ESD9B5.0ST5G
- added F401: 0.5A, Fuse:Fuse_1206_3216Metric, symbol Device:Polyfuse
- added F402: 1.1A, Fuse:Fuse_1812_4532Metric, symbol Device:Polyfuse
- added F403: 0.2A, Fuse:Fuse_1206_3216Metric, symbol Device:Polyfuse
- added J401: ESC1 CAN+PWM GH4, Connector_JST:JST_GH_SM04B-GHS-TB_1x04-1MP_P1.25mm_Horizontal, symbol Connector_Generic:Conn_01x04
- added J402: ESC2 CAN+PWM GH4, Connector_JST:JST_GH_SM04B-GHS-TB_1x04-1MP_P1.25mm_Horizontal, symbol Connector_Generic:Conn_01x04
- added J403: ESC3 CAN+PWM GH4, Connector_JST:JST_GH_SM04B-GHS-TB_1x04-1MP_P1.25mm_Horizontal, symbol Connector_Generic:Conn_01x04
- added J404: ESC4 CAN+PWM GH4, Connector_JST:JST_GH_SM04B-GHS-TB_1x04-1MP_P1.25mm_Horizontal, symbol Connector_Generic:Conn_01x04
- added J405: ESC5 CAN+PWM GH4, Connector_JST:JST_GH_SM04B-GHS-TB_1x04-1MP_P1.25mm_Horizontal, symbol Connector_Generic:Conn_01x04
- added J406: ESC6 CAN+PWM GH4, Connector_JST:JST_GH_SM04B-GHS-TB_1x04-1MP_P1.25mm_Horizontal, symbol Connector_Generic:Conn_01x04
- added J407: PM08-CAN GH4, Connector_JST:JST_GH_SM04B-GHS-TB_1x04-1MP_P1.25mm_Horizontal, symbol Connector_Generic:Conn_01x04
- added J408: BMS CAN GH4, Connector_JST:JST_GH_SM04B-GHS-TB_1x04-1MP_P1.25mm_Horizontal, symbol Connector_Generic:Conn_01x04
- added J409: REMOTE_ID GH4, Connector_JST:JST_GH_SM04B-GHS-TB_1x04-1MP_P1.25mm_Horizontal, symbol Connector_Generic:Conn_01x04
- added J410: GNSS2 (резерв) GH4, Connector_JST:JST_GH_SM04B-GHS-TB_1x04-1MP_P1.25mm_Horizontal, symbol Connector_Generic:Conn_01x04
- added J411: OBSTACLE_1 GH4, Connector_JST:JST_GH_SM04B-GHS-TB_1x04-1MP_P1.25mm_Horizontal, symbol Connector_Generic:Conn_01x04
- added J412: OBSTACLE_2 GH4, Connector_JST:JST_GH_SM04B-GHS-TB_1x04-1MP_P1.25mm_Horizontal, symbol Connector_Generic:Conn_01x04
- added J413: PRESSURE GH3, Connector_JST:JST_GH_SM03B-GHS-TB_1x03-1MP_P1.25mm_Horizontal, symbol Connector_Generic:Conn_01x03
- added J414: LEVEL GH3, Connector_JST:JST_GH_SM03B-GHS-TB_1x03-1MP_P1.25mm_Horizontal, symbol Connector_Generic:Conn_01x03
- added J415: FLOW GH3, Connector_JST:JST_GH_SM03B-GHS-TB_1x03-1MP_P1.25mm_Horizontal, symbol Connector_Generic:Conn_01x03
- added JP411: TERM_CAN1, Jumper:SolderJumper-2_P1.3mm_Open_RoundedPad1.0x1.5mm, symbol Jumper:SolderJumper_2_Open
- added JP421: TERM_CAN2, Jumper:SolderJumper-2_P1.3mm_Open_RoundedPad1.0x1.5mm, symbol Jumper:SolderJumper_2_Open
- added L411, L421: 744232090, Inductor_SMD:L_CommonMode_Wurth_WE-CNSW-1206, symbol Filter:Choke_Wurth_WE-CNSW_744232090
- added R411, R421: 120, Resistor_SMD:R_0805_2012Metric, symbol Device:R
- added R413, R423, R433, R434: 10k, Resistor_SMD:R_0402_1005Metric, symbol Device:R
- added R414, R424, R435: 20k, Resistor_SMD:R_0402_1005Metric, symbol Device:R
Connections:
- new net +12V: F402.1
- new net +5V: F401.1, F403.1
- new net ADC_LEVEL: C421.1, R423.2, R424.1
- new net ADC_PRESS: C411.1, R413.2, R414.1
- new net C1H: D411.1 (K), J401.2 (Pin_2), J402.2 (Pin_2), J403.2 (Pin_2), J404.2 (Pin_2), J405.2 (Pin_2), J406.2 (Pin_2), JP411.1 (A), L411.2
- new net C1L: D411.2 (K), J401.3 (Pin_3), J402.3 (Pin_3), J403.3 (Pin_3), J404.3 (Pin_3), J405.3 (Pin_3), J406.3 (Pin_3), L411.3, R411.2
- new net C1T: JP411.2 (B), R411.1
- new net C2H: D421.1 (K), J407.2 (Pin_2), J408.2 (Pin_2), J409.2 (Pin_2), J410.2 (Pin_2), J411.2 (Pin_2), J412.2 (Pin_2), JP421.1 (A), L421.2
- new net C2L: D421.2 (K), J407.3 (Pin_3), J408.3 (Pin_3), J409.3 (Pin_3), J410.3 (Pin_3), J411.3 (Pin_3), J412.3 (Pin_3), L421.3, R421.2
- new net C2T: JP421.2 (B), R421.1
- new net CAN1_H: L411.1
- new net CAN1_L: L411.4
- new net CAN2_H: L421.1
- new net CAN2_L: L421.4
- new net ESC_PWM1: J401.1 (Pin_1)
- new net ESC_PWM2: J402.1 (Pin_1)
- new net ESC_PWM3: J403.1 (Pin_1)
- new net ESC_PWM4: J404.1 (Pin_1)
- new net ESC_PWM5: J405.1 (Pin_1)
- new net ESC_PWM6: J406.1 (Pin_1)
- new net FLOW_CAP: C431.1, R434.2, R435.1
- new net FLOW_IN: D432.1 (A1), J415.2 (Pin_2), R433.2, R434.1
- new net GND: C411.2, C421.2, C431.2, D411.3 (A), D412.2 (A2), D421.3 (A), D422.2 (A2), D432.2 (A2), J401.4 (Pin_4), J402.4 (Pin_4), J403.4 (Pin_4), J404.4 (Pin_4), J405.4 (Pin_4), J406.4 (Pin_4), J407.4 (Pin_4), J408.4 (Pin_4), J409.4 (Pin_4), J410.4 (Pin_4), J411.4 (Pin_4), J412.4 (Pin_4), J413.3 (Pin_3), J414.3 (Pin_3), J415.3 (Pin_3), R414.2, R424.2, R435.2
- new net LEVEL_IN: D422.1 (A1), J414.2 (Pin_2), R423.1
- new net PRESS_IN: D412.1 (A1), J413.2 (Pin_2), R413.1
- new net V12_OBST: F402.2, J411.1 (Pin_1), J412.1 (Pin_1)
- new net V5_CAN2: F401.2, J409.1 (Pin_1), J410.1 (Pin_1)
- new net V5_SENS: F403.2, J413.1 (Pin_1), J414.1 (Pin_1), J415.1 (Pin_1), R433.1
- no-connect marks 0 -> 2
Other:
- note added: "CAN1: шесть ESC (DroneCAN) + резервный PWM в том же разъёме. CAN2: PM08-CAN, BMS, Remote ID, резервный GNSS, 2 радара препятствий. На каждой шине: синфазный дроссель L4x1 (WE-CNSW 744232090), ESD NUP2105L, терминатор 120 Ом через перемычку JP. JP замыкать только если плата — конец шины. ВНИМАНИЕ: кабели ESC ~0.9 м — это ответвления звезды; для 1 Мбит/с допустимы ~0.3 м. Решение (шлейф по лучам ил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"
- company: (none) -> АГД6.07.010
- title: (none) -> CAN_AND_SENSORS
Changed lines of the file:
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@@
-(kicad_sch
-	(version 20260306)
-	(generator "eeschema")
-	(generator_version "10.0")
-	(paper "A4")
-	(text "Grounding and cable shield termination defined at one point"
-		(exclude_from_sim no)
-		(at 20 71 0)
-		(effects
-			(font
-				(size 1.5 1.5)
-			)
-			(justify left bottom)
-		)
-	)
-	(text "Two protected CAN-FD branches with selectable termination"
-		(exclude_from_sim no)
-		(at 20 35 0)
-		(effects
-			(font
-				(size 1.5 1.5)
-			)
-			(justify left bottom)
-		)
-	)
-	(text "DATA_REQUIRED: sensor list, cable lengths and bus bit rate"
-		(exclude_from_sim no)
-		(at 20 83 0)
-		(effects
-			(font
-				(size 1.5 1.5)
-			)
-			(justify left bottom)
-		)
-	)
-	(text "Pressure, flow, tank level, temperature and obstacle interfaces"
-		(exclude_from_sim no)
-		(at 20 47 0)
-		(effects
-			(font
-				(size 1.5 1.5)
-			)
-			(justify left bottom)
-		)
-	)
-	(text "Per-branch power switching and fault telemetry"
-		(exclude_from_sim no)
-		(at 20 59 0)
-		(effects
-			(font
-				(size 1.5 1.5)
-			)
-			(justify left bottom)
-		)
-	)
-	(text "CAN_AND_SENSORS"
-		(exclude_from_sim no)
-		(at 20 20 0)
-		(effects
-			(font
-				(size 2.5 2.5)
-				(bold yes)
-			)
-			(justify left bottom)
-		)
-	)
-	(sheet_instances
-		(path "/"
-			(page "1")
-		)
-	)
-)

Commit message: AGD6.07.010 rev 0.3: design review fixes and bring-up plan
Design review (DESIGN_REVIEW.md) with fixes applied to the schematic:
INA228 input RC filters, 12 V bus current monitor (INA228 0x45),
BTS5030 diagnostic scaling with clamp diodes, flow input level fix,
CAN1 changed from star to daisy chain with on-board terminator, AI
shutdown request, board buzzer, series resistors and ESD on external
I2C probes. Connectors merged so every connector sits on a board edge.
Adds calculations.md (power, IPC-2221 widths, hot-swap, thermal, ADC
scaling, CAN, clearances) and BRINGUP.md (step-by-step test plan).
ERC: no errors; all 820 intended pin connections verified. Board is
re-placed; routing in progress.

Co-Authored-By: Claude Opus 5.5 <noreply@anthropic.com>
Claude-Session: https://claude.ai/code/session_01Qk7uTKdi6YbndB9fGuguYV
Parts:
- removed J403: ESC3 CAN+PWM GH4, Connector_JST:JST_GH_SM04B-GHS-TB_1x04-1MP_P1.25mm_Horizontal, symbol Connector_Generic:Conn_01x04
- removed J404: ESC4 CAN+PWM GH4, Connector_JST:JST_GH_SM04B-GHS-TB_1x04-1MP_P1.25mm_Horizontal, symbol Connector_Generic:Conn_01x04
- removed J405: ESC5 CAN+PWM GH4, Connector_JST:JST_GH_SM04B-GHS-TB_1x04-1MP_P1.25mm_Horizontal, symbol Connector_Generic:Conn_01x04
- removed J406: ESC6 CAN+PWM GH4, Connector_JST:JST_GH_SM04B-GHS-TB_1x04-1MP_P1.25mm_Horizontal, symbol Connector_Generic:Conn_01x04
- removed J413: PRESSURE GH3, Connector_JST:JST_GH_SM03B-GHS-TB_1x03-1MP_P1.25mm_Horizontal, symbol Connector_Generic:Conn_01x03
- removed J414: LEVEL GH3, Connector_JST:JST_GH_SM03B-GHS-TB_1x03-1MP_P1.25mm_Horizontal, symbol Connector_Generic:Conn_01x03
- removed J415: FLOW GH3, Connector_JST:JST_GH_SM03B-GHS-TB_1x03-1MP_P1.25mm_Horizontal, symbol Connector_Generic:Conn_01x03
- removed JP411: TERM_CAN1, Jumper:SolderJumper-2_P1.3mm_Open_RoundedPad1.0x1.5mm, symbol Jumper:SolderJumper_2_Open
- added D433: BAT54S, Package_TO_SOT_SMD:SOT-23, symbol Diode:BAT54S
- added J413: SPRAY_SENSORS GH8 (давл./уровень/расход), Connector_JST:JST_GH_SM08B-GHS-TB_1x08-1MP_P1.25mm_Horizontal, symbol Connector_Generic:Conn_01x08
- added J421: ESC1-6 PWM backup GH8, Connector_JST:JST_GH_SM08B-GHS-TB_1x08-1MP_P1.25mm_Horizontal, symbol Connector_Generic:Conn_01x08
- added JP411: TERM_CAN1 (замкнута), Jumper:SolderJumper-2_P1.3mm_Bridged_RoundedPad1.0x1.5mm, symbol Jumper:SolderJumper_2_Bridged
- J401: value ESC1 CAN+PWM GH4 -> CAN1 ESC CHAIN START GH4
- J402: value ESC2 CAN+PWM GH4 -> CAN1 ESC CHAIN RETURN GH4
- R435: value 20k -> 33k
Connections:
- net C1H: now also JP411.1 (A)
- net C1T: now also JP411.2 (B)
- net ESC_PWM1: now also J421.1 (Pin_1); no longer J401.1 (Pin_1)
- net ESC_PWM2: now also J421.2 (Pin_2); no longer J402.1 (Pin_1)
- net ESC_PWM3: now also J421.3 (Pin_3)
- net ESC_PWM4: now also J421.4 (Pin_4)
- net ESC_PWM5: now also J421.5 (Pin_5)
- net ESC_PWM6: now also J421.6 (Pin_6)
- net FLOW_CAP: now also D433.3 (COM)
- net FLOW_IN: now also J413.4 (Pin_4)
- net GND: now also D433.1 (A), J413.7 (Pin_7), J413.8 (Pin_8), J421.7 (Pin_7), J421.8 (Pin_8)
- net LEVEL_IN: now also J413.3 (Pin_3)
- net PRESS_IN: now also J413.2 (Pin_2)
- net V5_SENS: now also J413.1 (Pin_1), J413.5 (Pin_5), J413.6 (Pin_6)
- new net +3V3: D433.2 (K)
- no-connect marks 2 -> 4
Other:
- note added: "CAN1 (rev 0.3, DESIGN_REVIEW R12): ШЛЕЙФ — плата = начало шины (терминатор JP411 замкнут), J401 -> ESC1 -> ... -> ESC6 (терминатор на ESC6); J402 — резервный возврат шлейфа. Резервный PWM ESC1–6 — общий разъём J421 (GH8), жгут разветвляется по лучам. CAN2: PM08-CAN, BMS, Remote ID, резервный GNSS, 2 радара; ответвления <= 0.3 м, 500 кбит/с (R13). На каждой шине: синфазный дроссель L4x1 (WE-CNSW 7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"
- note removed: "CAN1: шесть ESC (DroneCAN) + резервный PWM в том же разъёме. CAN2: PM08-CAN, BMS, Remote ID, резервный GNSS, 2 радара препятствий. На каждой шине: синфазный дроссель L4x1 (WE-CNSW 744232090), ESD NUP2105L, терминатор 120 Ом через перемычку JP. JP замыкать только если плата — конец шины. ВНИМАНИЕ: кабели ESC ~0.9 м — это ответвления звезды; для 1 Мбит/с допустимы ~0.3 м. Решение (шлейф по лучам ил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"
