File: hardware/AGD6.07.010/flight_control_io.kicad_sch (KiCad schematic)
At the start: 0 parts

Commit message: Draw full AGD6.07.010 schematic per integrated_avionics_board spec
All ten sheets now carry components: 14S input with hot-swap and power
monitor, 12/5/3.3 V rails and a separate 12 V AI channel with soft-start
and current telemetry, Pixhawk connectors, CAN1/CAN2 hub with chokes,
ESD and switchable termination, sensor conditioning, SIYI and radar,
AI interface and watchdog, protected 12 V switches with diagnostics,
fan/heater control, cameras and Ethernet. Open choices are recorded in
DECISIONS.md; datasheet-dependent values are flagged CHECK_DATASHEET.

ERC: no errors. All 752 intended pin connections match the KiCad netlist.

Co-Authored-By: Claude Opus 5.5 <noreply@anthropic.com>
Claude-Session: https://claude.ai/code/session_01Qk7uTKdi6YbndB9fGuguYV
Parts:
- added D301, D302, D303, D304: ESD9B5.0ST5G, Diode_SMD:D_SOD-923, symbol Diode:ESD9B5.0ST5G
- added J301: PX_CAN1 GH4, Connector_JST:JST_GH_SM04B-GHS-TB_1x04-1MP_P1.25mm_Horizontal, symbol Connector_Generic:Conn_01x04
- added J302: PX_CAN2 GH4, Connector_JST:JST_GH_SM04B-GHS-TB_1x04-1MP_P1.25mm_Horizontal, symbol Connector_Generic:Conn_01x04
- added J303: PX_TELEM1 SIYI GH6, Connector_JST:JST_GH_SM06B-GHS-TB_1x06-1MP_P1.25mm_Horizontal, symbol Connector_Generic:Conn_01x06
- added J304: PX_TELEM2 AI GH6, Connector_JST:JST_GH_SM06B-GHS-TB_1x06-1MP_P1.25mm_Horizontal, symbol Connector_Generic:Conn_01x06
- added J305: PX_TELEM3 RADAR GH6, Connector_JST:JST_GH_SM06B-GHS-TB_1x06-1MP_P1.25mm_Horizontal, symbol Connector_Generic:Conn_01x06
- added J306: PX_I2C GH4, Connector_JST:JST_GH_SM04B-GHS-TB_1x04-1MP_P1.25mm_Horizontal, symbol Connector_Generic:Conn_01x04
- added J307: PX_AD&IO GH8, Connector_JST:JST_GH_SM08B-GHS-TB_1x08-1MP_P1.25mm_Horizontal, symbol Connector_Generic:Conn_01x08
- added J308: PX_RC_IN GH3, Connector_JST:JST_GH_SM03B-GHS-TB_1x03-1MP_P1.25mm_Horizontal, symbol Connector_Generic:Conn_01x03
- added J309: PX_MAIN 1-8, Connector_PinHeader_2.54mm:PinHeader_1x10_P2.54mm_Vertical, symbol Connector_Generic:Conn_01x10
- added J310: PX_AUX 1-8, Connector_PinHeader_2.54mm:PinHeader_1x10_P2.54mm_Vertical, symbol Connector_Generic:Conn_01x10
- added J311: FTS GH3, Connector_JST:JST_GH_SM03B-GHS-TB_1x03-1MP_P1.25mm_Horizontal, symbol Connector_Generic:Conn_01x03
- added J312: MODE_SWITCH GH4, Connector_JST:JST_GH_SM04B-GHS-TB_1x04-1MP_P1.25mm_Horizontal, symbol Connector_Generic:Conn_01x04
- added J313: LID_BATT_LATCH GH3, Connector_JST:JST_GH_SM03B-GHS-TB_1x03-1MP_P1.25mm_Horizontal, symbol Connector_Generic:Conn_01x03
- added R301: 100, Resistor_SMD:R_0402_1005Metric, symbol Device:R
- added R302, R303, R304, R307, R308: 1k, Resistor_SMD:R_0402_1005Metric, symbol Device:R
- added R305, R306, R309: 10k, Resistor_SMD:R_0402_1005Metric, symbol Device:R
- added R310, R311: 2.2k DNP, Resistor_SMD:R_0402_1005Metric, symbol Device:R
Connections:
- new net +3V3: R302.1, R307.1, R310.1, R311.1
- new net ADC_LEVEL: J307.3 (Pin_3)
- new net ADC_PRESS: J307.2 (Pin_2)
- new net AI_RX: J304.2 (Pin_2)
- new net AI_TX: J304.3 (Pin_3)
- new net CAM_TRIG: J310.7 (Pin_7)
- new net CAN1_H: J301.2 (Pin_2)
- new net CAN1_L: J301.3 (Pin_3)
- new net CAN2_H: J302.2 (Pin_2)
- new net CAN2_L: J302.3 (Pin_3)
- new net ENCL_C: D304.1 (A1), J313.2 (Pin_2), R308.1
- new net ENCL_COM: J313.1 (Pin_1), R307.2
- new net ENCL_OK: J307.7 (Pin_7), R308.2, R309.1
- new net ESC_PWM1: J309.1 (Pin_1)
- new net ESC_PWM2: J309.2 (Pin_2)
- new net ESC_PWM3: J309.3 (Pin_3)
- new net ESC_PWM4: J309.4 (Pin_4)
- new net ESC_PWM5: J309.5 (Pin_5)
- new net ESC_PWM6: J309.6 (Pin_6)
- new net FAN_CTL: J310.5 (Pin_5)
- new net FLOW_CAP: J307.4 (Pin_4)
- new net FTS_C: D301.1 (A1), J311.2 (Pin_2), R301.2
- new net FTS_TRIG: J309.7 (Pin_7), R301.1
- new net GND: D301.2 (A2), D302.2 (A2), D303.2 (A2), D304.2 (A2), J301.4 (Pin_4), J302.4 (Pin_4), J303.6 (Pin_6), J304.6 (Pin_6), J305.6 (Pin_6), J306.4 (Pin_4), J307.8 (Pin_8), J308.3 (Pin_3), J309.10 (Pin_10), J309.9 (Pin_9), J310.10 (Pin_10), J310.9 (Pin_9), J311.3 (Pin_3), J312.4 (Pin_4), J313.3 (Pin_3), R305.2, R306.2, R309.2
- new net HEATER_CTL: J310.6 (Pin_6)
- new net I2C_SCL: J306.2 (Pin_2), R310.2
- new net I2C_SDA: J306.3 (Pin_3), R311.2
- new net LIGHTS_CTL: J310.3 (Pin_3)
- new net MAV_PX_RX: J303.3 (Pin_3)
- new net MAV_PX_TX: J303.2 (Pin_2)
- new net MODE_A: J307.5 (Pin_5), R303.2, R305.1
- new net MODE_A_C: D302.1 (A1), J312.2 (Pin_2), R303.1
- new net MODE_B: J307.6 (Pin_6), R304.2, R306.1
- new net MODE_B_C: D303.1 (A1), J312.3 (Pin_3), R304.1
- new net MODE_COM: J312.1 (Pin_1), R302.2
- new net PUMP_PWM: J310.4 (Pin_4)
- new net RADAR_PX_RX: J305.3 (Pin_3)
- new net RADAR_PX_TX: J305.2 (Pin_2)
- new net SBUS: J308.2 (Pin_2)
- new net VALVE1_CTL: J310.1 (Pin_1)
- new net VALVE2_CTL: J310.2 (Pin_2)
- no-connect marks 0 -> 17
Other:
- note added: "R310/R311 не устанавливать: подтяжки I2C есть в Pixhawk. Установить, если шина работает без Pixhawk."
- note added: "РАЗЪЁМЫ К PIXHAWK 6X (распределение портов — DECISIONS.md). Pixhawk — единственный контур управления моторами. Выводы 5 V разъёмов Pixhawk не соединяются с шинами платы (NC, DECISIONS D17). Распиновки разъёмов Pixhawk — CHECK_DATASHEET (Pixhawk 6X / Pixhawk Connector Standard). MAIN1–6: резервные PWM ESC (основное управление — DroneCAN по CAN1). MAIN7: команда FTS. J1110 ПЕРЕКЛЮЧАТЕЛЬ РЕЖИМОВ MAN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"
- company: (none) -> АГД6.07.010
- title: (none) -> FLIGHT_CONTROL_IO
Changed lines of the file:
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@@
-(kicad_sch
-	(version 20260306)
-	(generator "eeschema")
-	(generator_version "10.0")
-	(paper "A4")
-	(text "RC input and emergency stop path bypass AI software"
-		(exclude_from_sim no)
-		(at 20 59 0)
-		(effects
-			(font
-				(size 1.5 1.5)
-			)
-			(justify left bottom)
-		)
-	)
-	(text "Dual CAN, UART telemetry, I2C/SPI service, GPIO and safety input"
-		(exclude_from_sim no)
-		(at 20 47 0)
-		(effects
-			(font
-				(size 1.5 1.5)
-			)
-			(justify left bottom)
-		)
-	)
-	(text "Autopilot remains independent of companion AI computer"
-		(exclude_from_sim no)
-		(at 20 35 0)
-		(effects
-			(font
-				(size 1.5 1.5)
-			)
-			(justify left bottom)
-		)
-	)
-	(text "FLIGHT_CONTROL_IO"
-		(exclude_from_sim no)
-		(at 20 20 0)
-		(effects
-			(font
-				(size 2.5 2.5)
-				(bold yes)
-			)
-			(justify left bottom)
-		)
-	)
-	(text "DATA_REQUIRED: exact Pixhawk model and connector pinout"
-		(exclude_from_sim no)
-		(at 20 83 0)
-		(effects
-			(font
-				(size 1.5 1.5)
-			)
-			(justify left bottom)
-		)
-	)
-	(text "ESD protection and keyed locking connectors"
-		(exclude_from_sim no)
-		(at 20 71 0)
-		(effects
-			(font
-				(size 1.5 1.5)
-			)
-			(justify left bottom)
-		)
-	)
-	(sheet_instances
-		(path "/"
-			(page "1")
-		)
-	)
-)

Commit message: AGD6.07.010 rev 0.3: design review fixes and bring-up plan
Design review (DESIGN_REVIEW.md) with fixes applied to the schematic:
INA228 input RC filters, 12 V bus current monitor (INA228 0x45),
BTS5030 diagnostic scaling with clamp diodes, flow input level fix,
CAN1 changed from star to daisy chain with on-board terminator, AI
shutdown request, board buzzer, series resistors and ESD on external
I2C probes. Connectors merged so every connector sits on a board edge.
Adds calculations.md (power, IPC-2221 widths, hot-swap, thermal, ADC
scaling, CAN, clearances) and BRINGUP.md (step-by-step test plan).
ERC: no errors; all 820 intended pin connections verified. Board is
re-placed; routing in progress.

Co-Authored-By: Claude Opus 5.5 <noreply@anthropic.com>
Claude-Session: https://claude.ai/code/session_01Qk7uTKdi6YbndB9fGuguYV
Parts:
- removed J312: MODE_SWITCH GH4, Connector_JST:JST_GH_SM04B-GHS-TB_1x04-1MP_P1.25mm_Horizontal, symbol Connector_Generic:Conn_01x04
- removed J313: LID_BATT_LATCH GH3, Connector_JST:JST_GH_SM03B-GHS-TB_1x03-1MP_P1.25mm_Horizontal, symbol Connector_Generic:Conn_01x03
- added J312: MODE_SWITCH + LID/BATT_LATCH GH6, Connector_JST:JST_GH_SM06B-GHS-TB_1x06-1MP_P1.25mm_Horizontal, symbol Connector_Generic:Conn_01x06
Connections:
- net ENCL_C: now also J312.5 (Pin_5)
- net ENCL_COM: now also J312.4 (Pin_4)
- net GND: now also J312.6 (Pin_6)
- net MODE_A_C: now also J312.2 (Pin_2)
- net MODE_B_C: now also J312.3 (Pin_3)
- net MODE_COM: now also J312.1 (Pin_1)
- net AI_SHDN_REQ: now reaches J309.8 (Pin_8)
- net BUZZER_CTL: now reaches J310.8 (Pin_8)
- no-connect marks 17 -> 15
Other:
- note added: "РАЗЪЁМЫ К PIXHAWK 6X (распределение портов — DECISIONS.md). Pixhawk — единственный контур управления моторами. Выводы 5 V разъёмов Pixhawk не соединяются с шинами платы (NC, DECISIONS D17). Распиновки разъёмов Pixhawk — CHECK_DATASHEET (Pixhawk 6X / Pixhawk Connector Standard). MAIN1–6: резервные PWM ESC (основное управление — DroneCAN по CAN1). MAIN7: команда FTS. MAIN8: запрос выключения ИИ. AU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"
- note removed: "РАЗЪЁМЫ К PIXHAWK 6X (распределение портов — DECISIONS.md). Pixhawk — единственный контур управления моторами. Выводы 5 V разъёмов Pixhawk не соединяются с шинами платы (NC, DECISIONS D17). Распиновки разъёмов Pixhawk — CHECK_DATASHEET (Pixhawk 6X / Pixhawk Connector Standard). MAIN1–6: резервные PWM ESC (основное управление — DroneCAN по CAN1). MAIN7: команда FTS. J1110 ПЕРЕКЛЮЧАТЕЛЬ РЕЖИМОВ MAN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"
