File: hardware/AGD6.07.010/power_conversion.kicad_sch (KiCad schematic)
At the start: 0 parts

Commit message: Draw full AGD6.07.010 schematic per integrated_avionics_board spec
All ten sheets now carry components: 14S input with hot-swap and power
monitor, 12/5/3.3 V rails and a separate 12 V AI channel with soft-start
and current telemetry, Pixhawk connectors, CAN1/CAN2 hub with chokes,
ESD and switchable termination, sensor conditioning, SIYI and radar,
AI interface and watchdog, protected 12 V switches with diagnostics,
fan/heater control, cameras and Ethernet. Open choices are recorded in
DECISIONS.md; datasheet-dependent values are flagged CHECK_DATASHEET.

ERC: no errors. All 752 intended pin connections match the KiCad netlist.

Co-Authored-By: Claude Opus 5.5 <noreply@anthropic.com>
Claude-Session: https://claude.ai/code/session_01Qk7uTKdi6YbndB9fGuguYV
Parts:
- added C201: DATA_REQUIRED, Capacitor_SMD:C_0402_1005Metric, symbol Device:C
- added C202: 3.3n, Capacitor_SMD:C_0402_1005Metric, symbol Device:C
- added C203: 4.7u 100V, Capacitor_SMD:C_1210_3225Metric, symbol Device:C
- added C204, C213: 22u 25V, Capacitor_SMD:C_1210_3225Metric, symbol Device:C
- added C205, C214: 100u 25V, Capacitor_SMD:CP_Elec_10x10.5, symbol Device:C_Polarized
- added C206: 10u 25V, Capacitor_SMD:C_0805_2012Metric, symbol Device:C
- added C207, C208: 22u 10V, Capacitor_SMD:C_0805_2012Metric, symbol Device:C
- added C209, C210: 1u, Capacitor_SMD:C_0603_1608Metric, symbol Device:C
- added C211: 10u, Capacitor_SMD:C_0805_2012Metric, symbol Device:C
- added C212: 10u 100V, Capacitor_SMD:C_1210_3225Metric, symbol Device:C
- added C215: 100n, Capacitor_SMD:C_0402_1005Metric, symbol Device:C
- added D202: SMAJ15A, Diode_SMD:D_SMA, symbol Diode:SMAJ15A
- added D203: BAT54WS, Diode_SMD:D_SOD-323, symbol Device:D_Schottky
- added D204: 12V, LED_SMD:LED_0603_1608Metric, symbol Device:LED
- added D205: 5V, LED_SMD:LED_0603_1608Metric, symbol Device:LED
- added D206: 3V3, LED_SMD:LED_0603_1608Metric, symbol Device:LED
- added F202: 3A 60V Littelfuse 0456003, Fuse:Fuse_Littelfuse-NANO2-451_453, symbol Device:Fuse
- added J202: AI_POWER_12V XT30, Connector_AMASS:AMASS_XT30PW-F_1x02_P2.50mm_Horizontal, symbol Connector_Generic:Conn_01x02
- added L201: 4.7u 5A, Inductor_SMD:L_Bourns_SRP1245A, symbol Device:L
- added L202: 2.2u 4A, Inductor_SMD:L_Bourns_SRP5030T, symbol Device:L
- added PS201: TRACO TEP 75-4812WI, symbol AGD6:DCDC_MODULE
- added PS202: DATA_REQUIRED изолир. 48V->12V >=100W, symbol AGD6:DCDC_MODULE
- added Q201: 40V N-MOSFET >=40A D2PAK (напр. IPB017N06N3), Package_TO_SOT_SMD:TO-263-2, symbol Transistor_FET:Q_NMOS_GDS
- added R201: 10, Resistor_SMD:R_0402_1005Metric, symbol Device:R
- added R202: 33k, Resistor_SMD:R_0402_1005Metric, symbol Device:R
- added R203, R207, R208, R211: 10k, Resistor_SMD:R_0402_1005Metric, symbol Device:R
- added R204: 47k, Resistor_SMD:R_0402_1005Metric, symbol Device:R
- added R205: 6.8k, Resistor_SMD:R_0402_1005Metric, symbol Device:R
- added R206: DATA_REQUIRED, Resistor_SMD:R_0402_1005Metric, symbol Device:R
- added R209, R210: 100k, Resistor_SMD:R_0402_1005Metric, symbol Device:R
- added R212: 3.3k, Resistor_SMD:R_0402_1005Metric, symbol Device:R
- added R213: 1k, Resistor_SMD:R_0402_1005Metric, symbol Device:R
- added RS201: 5m 1W, Resistor_SMD:R_2512_6332Metric, symbol Device:R
- added TP201: +12V, TestPoint:TestPoint_Pad_D1.5mm, symbol Connector:TestPoint
- added TP202: +5V, TestPoint:TestPoint_Pad_D1.5mm, symbol Connector:TestPoint
- added TP203: +3V3, TestPoint:TestPoint_Pad_D1.5mm, symbol Connector:TestPoint
- added TP204: V12_AI, TestPoint:TestPoint_Pad_D1.5mm, symbol Connector:TestPoint
- added TP205: AI_PGOOD, TestPoint:TestPoint_Pad_D1.5mm, symbol Connector:TestPoint
- added TP206: AI_ALERT_N, TestPoint:TestPoint_Pad_D1.5mm, symbol Connector:TestPoint
- added TP207: PG5, TestPoint:TestPoint_Pad_D1.5mm, symbol Connector:TestPoint
- added U201: TPS62133RGTR, Package_DFN_QFN:VQFN-16-1EP_3x3mm_P0.5mm_EP1.68x1.68mm_ThermalVias, symbol Regulator_Switching:TPS62133
- added U202: AP2112K-3.3TRG1, Package_TO_SOT_SMD:SOT-23-5, symbol Regulator_Linear:AP2112K-3.3
- added U203: LM5069MM-2, Package_SO:MSOP-10_3x3mm_P0.5mm, symbol Power_Management:LM5069MM-2
- added U204: INA228AIDGSR, Package_SO:TSSOP-10_3x3mm_P0.5mm, symbol Sensor_Energy:INA228
Connections:
- new net +12V: C204.1, C205.1, C206.1, PS201.4 (+VOUT), R209.1, R211.1, TP201.1, U201.10 (VIN), U201.11 (VIN), U201.12 (VIN)
- new net +3V3: C210.1, C211.1, C215.1, R207.1, R208.1, R213.1, TP203.1, U202.5 (VOUT), U204.2 (A0), U204.6 (VS)
- new net +5V: C207.1, C208.1, C209.1, L202.2, R210.1, R212.1, TP202.1, U201.14 (VOS), U202.1 (VIN), U202.3 (EN)
- new net AI_ALERT_N: R208.2, TP206.1, U204.3 (~{Alert})
- new net AI_GATE: Q201.1 (G), R201.2
- new net AI_GATE_DRV: R201.1, U203.10 (GATE)
- new net AI_OV: R204.2, R205.1, U203.4 (OVLO)
- new net AI_PGOOD: R207.2, TP205.1, U203.8 (PGD)
- new net AI_PWRLIM: R206.1, U203.7 (PWR)
- new net AI_PWR_EN: D203.1 (K)
- new net AI_SNS: Q201.2 (D), RS201.2, U203.1 (SENSE), U204.9 (Vin-)
- new net AI_TMR: C201.1, U203.6 (TIMER)
- new net AI_UV: D203.2 (A), R202.2, R203.1, U203.3 (UVLO)
- new net EN5: R209.2, U201.13 (EN)
- new net GND: C201.2, C202.2, C203.2, C204.2, C205.2, C206.2, C207.2, C208.2, C209.2, C210.2, C211.2, C212.2, C213.2, C214.2, C215.2, D202.2 (A2), D204.1 (K), D205.1 (K), D206.1 (K), J202.2 (Pin_2), PS201.2 (-VIN), PS201.6 (-VOUT), PS202.2 (-VIN), PS202.6 (-VOUT), R203.2, R205.2, R206.2, U201.15 (GND), U201.16 (GND), U201.17 (GND), U201.5 (FB), U201.6 (GND), U201.7 (FSW), U201.8 (DEF), U202.2 (GND), U203.5 (GND), U204.1 (A1), U204.7 (GND)
- new net I2C_SCL: U204.5 (SCL)
- new net I2C_SDA: U204.4 (SDA)
- new net LED_D204: D204.2 (A), R211.2
- new net LED_D205: D205.2 (A), R212.2
- new net LED_D206: D206.2 (A), R213.2
- new net PG5: R210.2, TP207.1, U201.4 (PG)
- new net SS5: C202.1, U201.9 (SS/TR)
- new net SW5: L202.1, U201.1 (SW), U201.2 (SW), U201.3 (SW)
- new net V12AI_RAW: C213.1, D202.1 (A1), PS202.4 (+VOUT), R202.1, R204.1, RS201.1, U203.2 (VIN), U204.10 (Vin+)
- new net V12_AI: C214.1, J202.1 (Pin_1), Q201.3 (S), TP204.1, U203.9 (OUT), U204.8 (Vbus)
- new net VIN_AI: F202.2, L201.1
- new net VIN_AI_F: C212.1, L201.2, PS202.1 (+VIN)
- new net VIN_PROT: C203.1, F202.1, PS201.1 (+VIN)
- no-connect marks 0 -> 5
Other:
- note added: "12 V АВИОНИКИ: PS201 TRACO TEP 75-4812WI (вход 18–75 V, 75 W). Минус выхода соединён с GND платы. 5 V: U201 TPS62133 от 12 V (3 A). 3.3 V: U202 AP2112K-3.3 от 5 V (600 mA). 12 V ИИ (ТЗ п. 5: отдельный изолированный канал до 8 A): F202 -> LC-фильтр L201/C212 -> PS202 (модель DATA_REQUIRED) -> TVS D202 -> шунт RS201 -> soft-start / ограничение тока U203 LM5069-2 + Q201 -> J202 XT30 к ИИ. Телеметрия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"
- company: (none) -> АГД6.07.010
- title: (none) -> POWER_CONVERSION
Changed lines of the file:
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@@
-(kicad_sch
-	(version 20260306)
-	(generator "eeschema")
-	(generator_version "10.0")
-	(paper "A4")
-	(text "Isolated/non-isolated pre-regulator: architecture selection pending"
-		(exclude_from_sim no)
-		(at 20 35 0)
-		(effects
-			(font
-				(size 1.5 1.5)
-			)
-			(justify left bottom)
-		)
-	)
-	(text "AI rail: dedicated protected output, swappable compute module"
-		(exclude_from_sim no)
-		(at 20 71 0)
-		(effects
-			(font
-				(size 1.5 1.5)
-			)
-			(justify left bottom)
-		)
-	)
-	(text "5 V rail: autopilot peripherals and interfaces"
-		(exclude_from_sim no)
-		(at 20 59 0)
-		(effects
-			(font
-				(size 1.5 1.5)
-			)
-			(justify left bottom)
-		)
-	)
-	(text "12 V rail: cameras, radio and auxiliary payload"
-		(exclude_from_sim no)
-		(at 20 47 0)
-		(effects
-			(font
-				(size 1.5 1.5)
-			)
-			(justify left bottom)
-		)
-	)
-	(text "DATA_REQUIRED: rail currents, ripple, hold-up and thermal limits"
-		(exclude_from_sim no)
-		(at 20 83 0)
-		(effects
-			(font
-				(size 1.5 1.5)
-			)
-			(justify left bottom)
-		)
-	)
-	(text "POWER_CONVERSION"
-		(exclude_from_sim no)
-		(at 20 20 0)
-		(effects
-			(font
-				(size 2.5 2.5)
-				(bold yes)
-			)
-			(justify left bottom)
-		)
-	)
-	(sheet_instances
-		(path "/"
-			(page "1")
-		)
-	)
-)

Commit message: Place all AGD6.07.010 parts on a 90x130 mm 4-layer board
Board outline 90 x 130 mm, M3 holes on the 50 x 110 mm pattern, GND
plane on In1. All 264 parts placed (net-driven: passives next to the
pins they serve, connectors along the edges, THT and power parts
first). Net classes for 14S, AI 12 V, 12 V and low-voltage rails plus a
same-footprint pad rule; DRC shows no errors besides unrouted nets.
Placeholder footprint for the two DC/DC bricks until models are chosen.

Co-Authored-By: Claude Opus 5.5 <noreply@anthropic.com>
Claude-Session: https://claude.ai/code/session_01Qk7uTKdi6YbndB9fGuguYV
Parts:
- PS201, PS202: footprint (none) -> AGD6:DCDC_2x1in_PLACEHOLDER

Commit message: AGD6.07.010 rev 0.3: design review fixes and bring-up plan
Design review (DESIGN_REVIEW.md) with fixes applied to the schematic:
INA228 input RC filters, 12 V bus current monitor (INA228 0x45),
BTS5030 diagnostic scaling with clamp diodes, flow input level fix,
CAN1 changed from star to daisy chain with on-board terminator, AI
shutdown request, board buzzer, series resistors and ESD on external
I2C probes. Connectors merged so every connector sits on a board edge.
Adds calculations.md (power, IPC-2221 widths, hot-swap, thermal, ADC
scaling, CAN, clearances) and BRINGUP.md (step-by-step test plan).
ERC: no errors; all 820 intended pin connections verified. Board is
re-placed; routing in progress.

Co-Authored-By: Claude Opus 5.5 <noreply@anthropic.com>
Claude-Session: https://claude.ai/code/session_01Qk7uTKdi6YbndB9fGuguYV
Parts:
- added C216, C217: 100n, Capacitor_SMD:C_0603_1608Metric, symbol Device:C
- added C218: 22u 25V, Capacitor_SMD:C_1210_3225Metric, symbol Device:C
- added C219: 100n, Capacitor_SMD:C_0402_1005Metric, symbol Device:C
- added R214, R215, R216, R217: 10, Resistor_SMD:R_0603_1608Metric, symbol Device:R
- added R218: 10k, Resistor_SMD:R_0402_1005Metric, symbol Device:R
- added RS202: 10m 1W, Resistor_SMD:R_2512_6332Metric, symbol Device:R
- added TP208: V12_ALERT_N, TestPoint:TestPoint_Pad_D1.5mm, symbol Connector:TestPoint
- added U205: INA228AIDGSR, Package_SO:TSSOP-10_3x3mm_P0.5mm, symbol Sensor_Energy:INA228
Connections:
- net +12V: now also R217.1, RS202.2, U205.8 (Vbus); no longer PS201.4 (+VOUT)
- net +3V3: now also C219.1, R218.1, U205.1 (A1), U205.2 (A0), U205.6 (VS)
- net AI_SNS: now also R215.1; no longer U204.9 (Vin-)
- net GND: now also C218.2, C219.2, U205.7 (GND)
- net I2C_SCL: now also U205.5 (SCL)
- net I2C_SDA: now also U205.4 (SDA)
- net V12AI_RAW: now also R214.1; no longer U204.10 (Vin+)
- new net INA2_N: C216.2, R215.2, U204.9 (Vin-)
- new net INA2_P: C216.1, R214.2, U204.10 (Vin+)
- new net INA3_N: C217.2, R217.2, U205.9 (Vin-)
- new net INA3_P: C217.1, R216.2, U205.10 (Vin+)
- new net V12_ALERT_N: R218.2, TP208.1, U205.3 (~{Alert})
- new net V12_RAW: C218.1, PS201.4 (+VOUT), R216.1, RS202.1

Commit message: AGD6.07.010: AI computer RK3588 - PS202 = TEP 75-4812WI, RS201 10 mOhm, docs and outputs updated
Co-Authored-By: Claude Opus 5.5 <noreply@anthropic.com>
Claude-Session: https://claude.ai/code/session_01Qk7uTKdi6YbndB9fGuguYV
Parts:
- PS202: value DATA_REQUIRED изолир. 48V->12V >=100W -> TRACO TEP 75-4812WI
- RS201: value 5m 1W -> 10m 1W
Other:
- note added: "12 V АВИОНИКИ: PS201 TRACO TEP 75-4812WI (вход 18–75 V, 75 W). Минус выхода соединён с GND платы. 5 V: U201 TPS62133 от 12 V (3 A). 3.3 V: U202 AP2112K-3.3 от 5 V (600 mA). 12 V ИИ (ТЗ п. 5, ИИ = RK3588, DECISIONS D18): F202 -> LC-фильтр L201/C212 -> PS202 TRACO TEP 75-4812WI (75 W, 6.25 A) -> TVS D202 -> шунт RS201 10 мОм (порог LM5069 ~5.5 A) -> soft-start / ограничение тока U203 LM5069-2 + Q20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"
- note removed: "12 V АВИОНИКИ: PS201 TRACO TEP 75-4812WI (вход 18–75 V, 75 W). Минус выхода соединён с GND платы. 5 V: U201 TPS62133 от 12 V (3 A). 3.3 V: U202 AP2112K-3.3 от 5 V (600 mA). 12 V ИИ (ТЗ п. 5: отдельный изолированный канал до 8 A): F202 -> LC-фильтр L201/C212 -> PS202 (модель DATA_REQUIRED) -> TVS D202 -> шунт RS201 -> soft-start / ограничение тока U203 LM5069-2 + Q201 -> J202 XT30 к ИИ. Телеметрия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"

Commit message: AGD6.07.010 rev 0.4 (WIP): 3x TRACO THL40 DC/DC, split 12 V bus, SwitchBlox Ethernet, fixed LM5069 UVLO/OVLO, computed hot-swap values, PX4 firmware notes; board re-placed, routing in progress
Co-Authored-By: Claude Opus 5.5 <noreply@anthropic.com>
Claude-Session: https://claude.ai/code/session_01Qk7uTKdi6YbndB9fGuguYV
Parts:
- removed PS201, PS202: TRACO TEP 75-4812WI, AGD6:DCDC_2x1in_PLACEHOLDER, symbol AGD6:DCDC_MODULE
- added C220: 22u 25V, Capacitor_SMD:C_1210_3225Metric, symbol Device:C
- added C221: 100u 25V, Capacitor_SMD:CP_Elec_10x10.5, symbol Device:C_Polarized
- added C222: 4.7u 100V, Capacitor_SMD:C_1210_3225Metric, symbol Device:C
- added D207: 12VA, LED_SMD:LED_0603_1608Metric, symbol Device:LED
- added PS201, PS202, PS203: TRACO THL 40-4812WI, Converter_DCDC:Converter_DCDC_TRACO_THL40-xxxxWI_THT, symbol AGD6:THL40-4812WI
- added R219: 10k, Resistor_SMD:R_0402_1005Metric, symbol Device:R
- added TP209: +12VA, TestPoint:TestPoint_Pad_D1.5mm, symbol Connector:TestPoint
- C201: value DATA_REQUIRED -> 220n; Note CHECK_DATASHEET -> РАСЧЁТ: calculations.md; Purpose (none) -> t_fault = C x 4 V / 85 uA = 10 ms
- R206: value DATA_REQUIRED -> 18.7k; Note CHECK_DATASHEET -> РАСЧЁТ: calculations.md; Purpose (none) -> P_LIM Q201 = 10 W: R = 1.25e5 x 0.015 x 10
- RS201: value 10m 1W -> 15m 1W; Note CHECK_DATASHEET -> РАСЧЁТ: calculations.md
Connections:
- net GND: now also C220.2, C221.2, C222.2, D207.1 (K), PS201.2 (-Vin), PS201.5 (-Vout), PS202.2 (-Vin), PS202.5 (-Vout), PS203.2 (-Vin), PS203.5 (-Vout)
- net V12AI_RAW: now also PS202.3 (+Vout)
- net V12_RAW: now also PS201.3 (+Vout)
- net VIN_AI_F: now also PS202.1 (+Vin)
- net VIN_PROT: now also C222.1, PS201.1 (+Vin), PS203.1 (+Vin)
- new net +12VA: C220.1, C221.1, PS203.3 (+Vout), R219.1, TP209.1
- new net LED_D207: D207.2 (A), R219.2
- no-connect marks 5 -> 7
Other:
- note added: "rev 0.4: ТРИ ИЗОЛИРОВАННЫХ МОДУЛЯ TRACO THL 40-4812WI (вход 18–75 V, 12 V / 3.35 A, 40 W, корпус 1"x1"; символ и посадочное место — библиотека KiCad 10). PS201 -> шина А +12V (SIYI, камеры, радары, SwitchBlox, 5 V, зуммер), телеметрия U205 INA228 0x45. PS203 -> шина Б +12VA (клапаны, огни, вентилятор, нагреватель), контроль напряжения — АЦП U804 (V12_MON). 5 V: U201 TPS62133 от +12V (3 A). 3.3 V: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"
- note added: "Изолированные DC/DC: 3 x TRACO THL 40-4812WI (шина А, шина Б, ИИ)"
- note removed: "12 V АВИОНИКИ: PS201 TRACO TEP 75-4812WI (вход 18–75 V, 75 W). Минус выхода соединён с GND платы. 5 V: U201 TPS62133 от 12 V (3 A). 3.3 V: U202 AP2112K-3.3 от 5 V (600 mA). 12 V ИИ (ТЗ п. 5, ИИ = RK3588, DECISIONS D18): F202 -> LC-фильтр L201/C212 -> PS202 TRACO TEP 75-4812WI (75 W, 6.25 A) -> TVS D202 -> шунт RS201 10 мОм (порог LM5069 ~5.5 A) -> soft-start / ограничение тока U203 LM5069-2 + Q20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"
- note removed: "Isolated/non-isolated pre-regulator: architecture selection pending"
